File: générateur de signal/générateur de signal/générateur_signal/Adressage.sch (KiCad schematic (older format))
At the start: 21 parts, among them SW1 SW_DIP_x01, SW2 SW_DIP_x01, U1 CD74HC4052PWR, U3 ATtiny84A-PU, U4 CD74HC4052PWR, U5 CD74HC4052PWR

Commit message: V3
+routage
Parts:
- D5, D6, D7, D8: footprint (none) -> LED_THT:LED_D3.0mm
- R10, R11, R12, R16, R17, R18, R19: footprint (none) -> Resistor_SMD:R_0805_2012Metric_Pad1.15x1.40mm_HandSolder
- R20, R21, R8, R9: renamed from R?; value R -> 10k; footprint (none) -> Resistor_SMD:R_0805_2012Metric_Pad1.15x1.40mm_HandSolder
- SW1, SW2: footprint (none) -> Connector_JST:JST_NV_B02P-NV_1x02_P5.00mm_Vertical
- U1, U4, U5: footprint SOP65P640X120-16N -> Empreintes:SOP65P640X120-16N
- U3: footprint Package_DIP:DIP-14_W7.62mm -> Package_DIP:DIP-14_W7.62mm_LongPads
Changed lines of the file:
@@
 F 0 "U3" H 4370 5596 50  0000 R CNN
 F 1 "ATtiny84A-PU" H 4370 5505 50  0000 R CNN
-F 2 "Package_DIP:DIP-14_W7.62mm" H 4900 5550 50  0001 C CIN
+F 2 "Package_DIP:DIP-14_W7.62mm_LongPads" H 4900 5550 50  0001 C CIN
 F 3 "http://ww1.microchip.com/downloads/en/DeviceDoc/doc8183.pdf" H 4900 5550 50  0001 C CNN
 	1    4900 5550
@@
 F 0 "SW2" V 2554 5680 50  0000 L CNN
 F 1 "SW_DIP_x01" V 2645 5680 50  0000 L CNN
-F 2 "" H 2600 5550 50  0001 C CNN
+F 2 "Connector_JST:JST_NV_B02P-NV_1x02_P5.00mm_Vertical" H 2600 5550 50  0001 C CNN
 F 3 "" H 2600 5550 50  0001 C CNN
 	1    2600 5550
@@
 F 0 "R11" H 3070 5796 50  0000 L CNN
 F 1 "56" H 3070 5705 50  0000 L CNN
-F 2 "" V 2930 5750 50  0001 C CNN
+F 2 "Resistor_SMD:R_0805_2012Metric_Pad1.15x1.40mm_HandSolder" V 2930 5750 50  0001 C CNN
 F 3 "~" H 3000 5750 50  0001 C CNN
 	1    3000 5750
@@
 F 0 "SW1" V 2554 5380 50  0000 L CNN
 F 1 "SW_DIP_x01" V 2645 5380 50  0000 L CNN
-F 2 "" H 2600 5250 50  0001 C CNN
+F 2 "Connector_JST:JST_NV_B02P-NV_1x02_P5.00mm_Vertical" H 2600 5250 50  0001 C CNN
 F 3 "" H 2600 5250 50  0001 C CNN
 	1    2600 5250
@@
 F 0 "U1" H 2950 4120 50  0000 C CNN
 F 1 "CD74HC4052PWR" H 2950 4029 50  0000 C CNN
-F 2 "SOP65P640X120-16N" H 2950 3150 50  0001 L BNN
+F 2 "Empreintes:SOP65P640X120-16N" H 2950 3150 50  0001 L BNN
 F 3 "TSSOP-16" H 2950 3150 50  0001 L BNN
 F 4 "-" H 2950 3150 50  0001 L BNN "Champ4"
@@
 F 0 "U4" H 4950 4120 50  0000 C CNN
 F 1 "CD74HC4052PWR" H 4950 4029 50  0000 C CNN
-F 2 "SOP65P640X120-16N" H 4950 3150 50  0001 L BNN
+F 2 "Empreintes:SOP65P640X120-16N" H 4950 3150 50  0001 L BNN
 F 3 "TSSOP-16" H 4950 3150 50  0001 L BNN
 F 4 "-" H 4950 3150 50  0001 L BNN "Champ4"
@@
 F 0 "U5" H 6950 4120 50  0000 C CNN
 F 1 "CD74HC4052PWR" H 6950 4029 50  0000 C CNN
-F 2 "SOP65P640X120-16N" H 6950 3150 50  0001 L BNN
+F 2 "Empreintes:SOP65P640X120-16N" H 6950 3150 50  0001 L BNN
 F 3 "TSSOP-16" H 6950 3150 50  0001 L BNN
 F 4 "-" H 6950 3150 50  0001 L BNN "Champ4"
@@
 F 0 "R10" H 3070 5146 50  0000 L CNN
 F 1 "56" H 3070 5055 50  0000 L CNN
-F 2 "" V 2930 5100 50  0001 C CNN
+F 2 "Resistor_SMD:R_0805_2012Metric_Pad1.15x1.40mm_HandSolder" V 2930 5100 50  0001 C CNN
 F 3 "~" H 3000 5100 50  0001 C CNN
 	1    3000 5100
@@
 F 0 "D5" V 8238 2883 50  0000 R CNN
 F 1 "LED" V 8147 2883 50  0000 R CNN
-F 2 "" H 8200 3000 50  0001 C CNN
+F 2 "LED_THT:LED_D3.0mm" H 8200 3000 50  0001 C CNN
 F 3 "~" H 8200 3000 50  0001 C CNN
 	1    8200 3000
@@
 F 0 "D6" V 8638 2783 50  0000 R CNN
 F 1 "LED" V 8547 2783 50  0000 R CNN
-F 2 "" H 8600 2900 50  0001 C CNN
+F 2 "LED_THT:LED_D3.0mm" H 8600 2900 50  0001 C CNN
 F 3 "~" H 8600 2900 50  0001 C CNN
 	1    8600 2900
@@
 F 0 "D7" V 8988 2683 50  0000 R CNN
 F 1 "LED" V 8897 2683 50  0000 R CNN
-F 2 "" H 8950 2800 50  0001 C CNN
+F 2 "LED_THT:LED_D3.0mm" H 8950 2800 50  0001 C CNN
 F 3 "~" H 8950 2800 50  0001 C CNN
 	1    8950 2800
@@
 F 0 "D8" V 9338 2583 50  0000 R CNN
 F 1 "LED" V 9247 2583 50  0000 R CNN
-F 2 "" H 9300 2700 50  0001 C CNN
+F 2 "LED_THT:LED_D3.0mm" H 9300 2700 50  0001 C CNN
 F 3 "~" H 9300 2700 50  0001 C CNN
 	1    9300 2700
@@
 F 0 "R12" H 3820 2296 50  0000 L CNN
 F 1 "10k" H 3820 2205 50  0000 L CNN
-F 2 "" V 3680 2250 50  0001 C CNN
+F 2 "Resistor_SMD:R_0805_2012Metric_Pad1.15x1.40mm_HandSolder" V 3680 2250 50  0001 C CNN
 F 3 "~" H 3750 2250 50  0001 C CNN
 	1    3750 2250
@@
 F 0 "R16" V 4300 2950 50  0000 C CNN
 F 1 "10k" V 4200 2950 50  0000 C CNN
-F 2 "" V 4030 3050 50  0001 C CNN
+F 2 "Resistor_SMD:R_0805_2012Metric_Pad1.15x1.40mm_HandSolder" V 4030 3050 50  0001 C CNN
 F 3 "~" H 4100 3050 50  0001 C CNN
 	1    4100 3050
@@
 F 0 "R17" H 5870 2146 50  0000 L CNN
 F 1 "10k" H 5870 2055 50  0000 L CNN
-F 2 "" V 5730 2100 50  0001 C CNN
+F 2 "Resistor_SMD:R_0805_2012Metric_Pad1.15x1.40mm_HandSolder" V 5730 2100 50  0001 C CNN
 F 3 "~" H 5800 2100 50  0001 C CNN
 	1    5800 2100
@@
 F 0 "R18" H 7920 3246 50  0000 L CNN
 F 1 "56" H 7920 3155 50  0000 L CNN
-F 2 "" V 7780 3200 50  0001 C CNN
+F 2 "Resistor_SMD:R_0805_2012Metric_Pad1.15x1.40mm_HandSolder" V 7780 3200 50  0001 C CNN
 F 3 "~" H 7850 3200 50  0001 C CNN
 	1    7850 3200
@@
 F 0 "R19" H 7920 3596 50  0000 L CNN
 F 1 "56" H 7920 3505 50  0000 L CNN
-F 2 "" V 7780 3550 50  0001 C CNN
+F 2 "Resistor_SMD:R_0805_2012Metric_Pad1.15x1.40mm_HandSolder" V 7780 3550 50  0001 C CNN
 F 3 "~" H 7850 3550 50  0001 C CNN
 	1    7850 3550
@@
 	7850 3700 7850 3850
 $Comp
-L Device:R R?
+L Device:R R21
 U 1 1 5EA60413
 P 4900 4800
-F 0 "R?" H 4970 4846 50  0000 L CNN
-F 1 "R" H 4970 4755 50  0000 L CNN
-F 2 "" V 4830 4800 50  0001 C CNN
+F 0 "R21" H 5050 4850 50  0000 L CNN
+F 1 "10k" H 5050 4750 50  0000 L CNN
+F 2 "Resistor_SMD:R_0805_2012Metric_Pad1.15x1.40mm_HandSolder" V 4830 4800 50  0001 C CNN
 F 3 "~" H 4900 4800 50  0001 C CNN
 	1    4900 4800
@@
 $EndComp
 $Comp
-L Device:R R?
+L Device:R R20
 U 1 1 5EA604C1
 P 4800 4800
-F 0 "R?" H 4870 4846 50  0000 L CNN
-F 1 "R" H 4870 4755 50  0000 L CNN
-F 2 "" V 4730 4800 50  0001 C CNN
+F 0 "R20" H 4600 4950 50  0000 L CNN
+F 1 "10k" H 4600 4850 50  0000 L CNN
+F 2 "Resistor_SMD:R_0805_2012Metric_Pad1.15x1.40mm_HandSolder" V 4730 4800 50  0001 C CNN
 F 3 "~" H 4800 4800 50  0001 C CNN
 	1    4800 4800
@@
 $EndComp
 $Comp
-L Device:R R?
+L Device:R R8
 U 1 1 5EA605FE
 P 4150 4900
-F 0 "R?" V 3943 4900 50  0000 C CNN
-F 1 "R" V 4034 4900 50  0000 C CNN
-F 2 "" V 4080 4900 50  0001 C CNN
+F 0 "R8" V 3943 4900 50  0000 C CNN
+F 1 "10k" V 4034 4900 50  0000 C CNN
+F 2 "Resistor_SMD:R_0805_2012Metric_Pad1.15x1.40mm_HandSolder" V 4080 4900 50  0001 C CNN
 F 3 "~" H 4150 4900 50  0001 C CNN
 	1    4150 4900
@@
 $EndComp
 $Comp
-L Device:R R?
+L Device:R R9
 U 1 1 5EA60683
 P 4250 4750
-F 0 "R?" V 4043 4750 50  0000 C CNN
-F 1 "R" V 4134 4750 50  0000 C CNN
-F 2 "" V 4180 4750 50  0001 C CNN
+F 0 "R9" V 4043 4750 50  0000 C CNN
+F 1 "10k" V 4134 4750 50  0000 C CNN
+F 2 "Resistor_SMD:R_0805_2012Metric_Pad1.15x1.40mm_HandSolder" V 4180 4750 50  0001 C CNN
 F 3 "~" H 4250 4750 50  0001 C CNN
 	1    4250 4750
@@
 	4700 4650 4700 4750
 $Comp
-L power:GND #PWR?
+L power:GND #PWR0130
 U 1 1 5EA6CB3E
 P 4700 4750
-F 0 "#PWR?" H 4700 4500 50  0001 C CNN
+F 0 "#PWR0130" H 4700 4500 50  0001 C CNN
 F 1 "GND" H 4705 4577 50  0000 C CNN
 F 2 "" H 4700 4750 50  0001 C CNN
@@
 Connection ~ 4000 4900
 $Comp
-L power:GND #PWR?
+L power:GND #PWR0131
 U 1 1 5EA7231C
 P 4000 5050
-F 0 "#PWR?" H 4000 4800 50  0001 C CNN
+F 0 "#PWR0131" H 4000 4800 50  0001 C CNN
 F 1 "GND" H 4005 4877 50  0000 C CNN
 F 2 "" H 4000 5050 50  0001 C CNN
