File: générateur de signal/générateur de signal/générateur_signal/Alimentation.sch (KiCad schematic (older format))
At the start: 7 parts, among them J3 Conn_Coaxial_Power

Commit message: V3
+routage
Parts:
- D1: renamed from D?; footprint (none) -> Empreintes:Zenner 5v
- D2: footprint (none) -> Empreintes:Zenner 5v
- D3, D4: footprint (none) -> Diode_SMD:D_SMA_Handsoldering
- J3: footprint (none) -> Connector_JST:JST_NV_B02P-NV_1x02_P5.00mm_Vertical
- R4: footprint (none) -> Resistor_THT:R_Axial_DIN0309_L9.0mm_D3.2mm_P12.70mm_Horizontal
- R5: renamed from R?; footprint (none) -> Resistor_THT:R_Axial_DIN0309_L9.0mm_D3.2mm_P12.70mm_Horizontal
Connections:
- wire segments 37 -> 35
Changed lines of the file:
@@
 F 0 "D2" V 7954 3329 50  0000 L CNN
 F 1 "5.1" V 8045 3329 50  0000 L CNN
-F 2 "" H 8000 3250 50  0001 C CNN
+F 2 "Empreintes:Zenner 5v" H 8000 3250 50  0001 C CNN
 F 3 "~" H 8000 3250 50  0001 C CNN
 	1    8000 3250
@@
 F 0 "D4" V 8004 2529 50  0000 L CNN
 F 1 "12" V 8095 2529 50  0000 L CNN
-F 2 "" H 8050 2450 50  0001 C CNN
+F 2 "Diode_SMD:D_SMA_Handsoldering" H 8050 2450 50  0001 C CNN
 F 3 "~" H 8050 2450 50  0001 C CNN
 	1    8050 2450
@@
 F 0 "D3" V 8004 1579 50  0000 L CNN
 F 1 "12" V 8095 1579 50  0000 L CNN
-F 2 "" H 8050 1500 50  0001 C CNN
+F 2 "Diode_SMD:D_SMA_Handsoldering" H 8050 1500 50  0001 C CNN
 F 3 "~" H 8050 1500 50  0001 C CNN
 	1    8050 1500
@@
 Text GLabel 8300 1450 3    50   Input ~ 0
 gbf2
-Wire Wire Line
-	8300 2300 8300 2400
 $Comp
 L Connector:Conn_Coaxial_Power J3
@@
 F 0 "J3" V 5183 2250 50  0000 C CNN
 F 1 "Conn_Coaxial_Power" V 5274 2250 50  0000 C CNN
-F 2 "" H 5400 2250 50  0001 C CNN
+F 2 "Connector_JST:JST_NV_B02P-NV_1x02_P5.00mm_Vertical" H 5400 2250 50  0001 C CNN
 F 3 "~" H 5400 2250 50  0001 C CNN
 	1    5400 2300
@@
 	4950 2150 4950 2300
 Wire Wire Line
-	4950 2300 5000 2300
-Wire Wire Line
 	5900 2300 5900 2350
 $Comp
@@
 	8300 1400 8300 1450
 $Comp
-L power:PWR_FLAG #FLG0102
-U 1 1 5E96DA55
-P 8300 2300
-F 0 "#FLG0102" H 8300 2375 50  0001 C CNN
-F 1 "PWR_FLAG" V 8300 2428 50  0000 L CNN
-F 2 "" H 8300 2300 50  0001 C CNN
-F 3 "~" H 8300 2300 50  0001 C CNN
-	1    8300 2300
-	0    1    1    0
-$EndComp
-$Comp
 L power:PWR_FLAG #FLG0104
 U 1 1 5E96DA64
@@
 $EndComp
 $Comp
-L power:PWR_FLAG #FLG0105
-U 1 1 5E96DA6B
-P 5000 2300
-F 0 "#FLG0105" H 5000 2375 50  0001 C CNN
-F 1 "PWR_FLAG" H 5000 2473 50  0000 C CNN
-F 2 "" H 5000 2300 50  0001 C CNN
-F 3 "~" H 5000 2300 50  0001 C CNN
-	1    5000 2300
-	-1   0    0    1
-$EndComp
-Connection ~ 5000 2300
-Wire Wire Line
-	5000 2300 5300 2300
-$Comp
 L power:GND #PWR0115
 U 1 1 5E96DA73
@@
 	8050 1650 8050 1700
 Wire Wire Line
-	8300 2150 8300 2300
-Connection ~ 8300 2300
-Wire Wire Line
 	8050 2300 8050 2150
 Connection ~ 8050 2150
@@
 F 0 "R4" V 7493 3050 50  0000 C CNN
 F 1 "1k" V 7584 3050 50  0000 C CNN
-F 2 "" V 7630 3050 50  0001 C CNN
+F 2 "Resistor_THT:R_Axial_DIN0309_L9.0mm_D3.2mm_P12.70mm_Horizontal" V 7630 3050 50  0001 C CNN
 F 3 "~" H 7700 3050 50  0001 C CNN
 	1    7700 3050
@@
 	7250 2150 8050 2150
 $Comp
-L Device:D_Zener D?
+L Device:D_Zener D1
 U 1 1 5E96014A
 P 8000 4050
-F 0 "D?" V 7954 4129 50  0000 L CNN
+F 0 "D1" V 7954 4129 50  0000 L CNN
 F 1 "5.1" V 8045 4129 50  0000 L CNN
-F 2 "" H 8000 4050 50  0001 C CNN
+F 2 "Empreintes:Zenner 5v" H 8000 4050 50  0001 C CNN
 F 3 "~" H 8000 4050 50  0001 C CNN
 	1    8000 4050
@@
 	8300 4000 8300 3900
 $Comp
-L power:PWR_FLAG #FLG?
+L power:PWR_FLAG #FLG0103
 U 1 1 5E960152
 P 8400 3900
-F 0 "#FLG?" H 8400 3975 50  0001 C CNN
+F 0 "#FLG0103" H 8400 3975 50  0001 C CNN
 F 1 "PWR_FLAG" V 8400 4028 50  0000 L CNN
 F 2 "" H 8400 3900 50  0001 C CNN
@@
 Connection ~ 8300 3900
 $Comp
-L Device:R R?
+L Device:R R5
 U 1 1 5E96015D
 P 7700 3850
-F 0 "R?" V 7493 3850 50  0000 C CNN
+F 0 "R5" V 7493 3850 50  0000 C CNN
 F 1 "470" V 7584 3850 50  0000 C CNN
-F 2 "" V 7630 3850 50  0001 C CNN
+F 2 "Resistor_THT:R_Axial_DIN0309_L9.0mm_D3.2mm_P12.70mm_Horizontal" V 7630 3850 50  0001 C CNN
 F 3 "~" H 7700 3850 50  0001 C CNN
 	1    7700 3850
@@
 Connection ~ 8000 3850
 $Comp
-L power:GND #PWR?
+L power:GND #PWR0119
 U 1 1 5E960165
 P 8000 4250
-F 0 "#PWR?" H 8000 4000 50  0001 C CNN
+F 0 "#PWR0119" H 8000 4000 50  0001 C CNN
 F 1 "GND" H 8005 4077 50  0000 C CNN
 F 2 "" H 8000 4250 50  0001 C CNN
@@
 Wire Wire Line
 	7250 1250 8050 1250
+Wire Wire Line
+	8300 2150 8300 2400
+Wire Wire Line
+	4950 2300 5300 2300
 $EndSCHEMATC
