File: générateur de signal/générateur de signal/générateur_signal/générateur_signal.sch (KiCad schematic (older format))
At the start: 56 parts, among them J1 Conn_Coaxial, J2 Conn_Coaxial, J3 Conn_Coaxial_Power, J4 Conn_Coaxial, J5 Conn_Coaxial, SW1 SW_DIP_x01, SW2 SW_DIP_x01, U1 CD74HC4052PWR, U2 XR2206CP-F, U3 ATtiny84A-PU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

Commit message: V2
+ ergonomie schéma
+ correction Zenner
Parts:
- removed D1, D2: 5.1, symbol Device:D_Zener
- removed D3, D4: 12, symbol Device:D_Zener
- removed D5, D6, D7, D8: LED, symbol Device:LED
- removed J3: Conn_Coaxial_Power, symbol Connector:Conn_Coaxial_Power
- removed R10, R8, R9: 10k, symbol Device:R
- removed R11, R12, R4, R5: 56, symbol Device:R
- removed SW1, SW2: SW_DIP_x01, symbol Switch:SW_DIP_x01
- removed U1, U4, U5: CD74HC4052PWR, SOP65P640X120-16N, symbol CD74HC4052PWR:CD74HC4052PWR
- removed U3: ATtiny84A-PU, Package_DIP:DIP-14_W7.62mm, symbol MCU_Microchip_ATtiny:ATtiny84A-PU
- added C11, C12, C13, C14, C15, C16, C17: 100n, symbol Device:C
Connections:
- net labels removed: +12V
- wire segments 264 -> 166
Other:
- moved on the sheet: U7

Commit message: V3
+routage
Parts:
- added C18, C19, C22, C23: 0.1u, Capacitor_SMD:C_0805_2012Metric_Pad1.15x1.40mm_HandSolder, symbol Device:C
- added C20, C21: 1u, Capacitor_SMD:C_0805_2012Metric_Pad1.15x1.40mm_HandSolder, symbol Device:C
- C1, C3: value 2,2u -> 1u; footprint (none) -> Capacitor_SMD:C_0805_2012Metric_Pad1.15x1.40mm_HandSolder
- C10: footprint (none) -> Capacitor_THT:CP_Radial_D6.3mm_P2.50mm
- C11, C12, C13, C14, C15, C16, C17, C2, C5, C6, C7, C8: footprint (none) -> Capacitor_SMD:C_0805_2012Metric_Pad1.15x1.40mm_HandSolder
- C4: footprint (none) -> Empreintes:2.2uF B(Size) Electrolytic
- C9: footprint (none) -> Capacitor_THT:CP_Radial_D5.0mm_P2.00mm
- J1, J2, J4, J5: footprint (none) -> Connector_JST:JST_NV_B02P-NV_1x02_P5.00mm_Vertical
- R1, R13, R14, R15, R2, R3, R6, R7: footprint (none) -> Resistor_SMD:R_0805_2012Metric_Pad1.15x1.40mm_HandSolder
- RV1, RV3, RV5, RV6, RV7: footprint (none) -> Empreintes:RM065
- RV2: value R_POT -> 10k; footprint (none) -> Empreintes:RM065
- RV4, RV8, RV9: footprint (none) -> Connector_PinHeader_2.54mm:PinHeader_1x03_P2.54mm_Vertical
- U2: footprint DIP254P762X533-16 -> Package_DIP:DIP-16_W7.62mm_LongPads
- U6: footprint SOIC127P600X175-8N -> Empreintes:SOIC127P600X175-8N
- U7: footprint (none) -> Package_DIP:DIP-8_W7.62mm_LongPads
Connections:
- wire segments 166 -> 182
